Commit message: scripts to use mocap data

File: model/urdf/4279_scaled.urdf (robot description, URDF)
Before this commit: robot 4279_scaled.urdf, 82 links, 81 joints
Links:
- link BHD: geometry visual sphere radius=0.02
- link C7_study: geometry visual sphere radius=0.02
- link FHD: geometry visual sphere radius=0.02
- link L.ASIS_study: geometry visual sphere radius=0.02
- link L.PSIS_study: geometry visual sphere radius=0.02
- link LHD: geometry visual sphere radius=0.02
- link LHL2: geometry visual sphere radius=0.02
- link LHM5: geometry visual sphere radius=0.02
- link L_5meta_study: geometry visual sphere radius=0.02
- link L_ankle_study: geometry visual sphere radius=0.02
- link L_calc_study: geometry visual sphere radius=0.02
- link L_knee_study: geometry visual sphere radius=0.02
- link L_lelbow_study: geometry visual sphere radius=0.02
- link L_lwrist_study: geometry visual sphere radius=0.02
- link L_mankle_study: geometry visual sphere radius=0.02
- link L_melbow_study: geometry visual sphere radius=0.02
- link L_mknee_study: geometry visual sphere radius=0.02
- link L_mwrist_study: geometry visual sphere radius=0.02
- link L_sh1_study: geometry visual sphere radius=0.02
- link L_shoulder_study: geometry visual sphere radius=0.02
- link L_thigh1_study: geometry visual sphere radius=0.02
- link L_toe_study: geometry visual sphere radius=0.02
- link RHD: geometry visual sphere radius=0.02
- link RHL2: geometry visual sphere radius=0.02
- link RHM5: geometry visual sphere radius=0.02
- link SJN: geometry visual sphere radius=0.02
- link STRN: geometry visual sphere radius=0.02
- link TV12: geometry visual sphere radius=0.02
- link TV8: geometry visual sphere radius=0.02
- link left_foot: geometry visual mesh filename=meshes/foot_mesh.STL scale=0.006700 0.006700 0.006700
- link left_hand: geometry visual mesh filename=meshes/hand_mesh.STL scale=0.006100 0.006100 0.006100
- link left_lowerarm: geometry visual mesh filename=meshes/elbow_mesh.STL scale=0.005500 0.005500 0.005500; visual mesh filename=meshes/lowerarm_mesh.STL scale=0.006400 0.006400 0.006400
- link left_lowerleg: geometry visual mesh filename=meshes/knee_mesh.STL scale=0.005600 0.005600 0.005600; visual mesh filename=meshes/lowerleg_mesh.STL scale=0.006300 0.006600 0.007000
- link left_upperarm: geometry visual mesh filename=meshes/shoulder_mesh.STL scale=0.003900 0.003900 0.003900; visual mesh filename=meshes/upperarm_mesh.STL scale=0.006300 0.006000 0.006900
- link left_upperleg: geometry visual mesh filename=meshes/upperleg_mesh.STL scale=0.006200 0.006400 0.006900
- link middle_abdomen: geometry visual mesh filename=meshes/abdomen_mesh.STL scale=0.007400 0.007400 0.007400
- link middle_head: geometry visual mesh filename=meshes/head_mesh.STL scale=0.005600 0.005600 0.005600; visual mesh filename=meshes/neck_mesh.STL scale=0.005000 0.005000 0.005000
- link middle_pelvis: geometry visual mesh filename=meshes/pelvis_mesh.STL scale=0.006300 0.005800 0.005800
- link middle_thorax: geometry visual mesh filename=meshes/torso_mesh.STL scale=0.007000 0.007000 0.007000
- link r.ASIS_study: geometry visual sphere radius=0.02
- link r.PSIS_study: geometry visual sphere radius=0.02
- link r_5meta_study: geometry visual sphere radius=0.02
- link r_ankle_study: geometry visual sphere radius=0.02
- link r_calc_study: geometry visual sphere radius=0.02
- link r_knee_study: geometry visual sphere radius=0.02
- link r_lelbow_study: geometry visual sphere radius=0.02
- link r_lwrist_study: geometry visual sphere radius=0.02
- link r_mankle_study: geometry visual sphere radius=0.02
- link r_melbow_study: geometry visual sphere radius=0.02
- link r_mknee_study: geometry visual sphere radius=0.02
- link r_mwrist_study: geometry visual sphere radius=0.02
- link r_sh1_study: geometry visual sphere radius=0.02
- link r_shoulder_study: geometry visual sphere radius=0.02
- link r_thigh1_study: geometry visual sphere radius=0.02
- link r_toe_study: geometry visual sphere radius=0.02
- link right_foot: geometry visual mesh filename=meshes/foot_mesh.STL scale=0.006700 0.006700 0.006700
- link right_hand: geometry visual mesh filename=meshes/hand_mesh.STL scale=0.006100 0.006100 0.006100
- link right_lowerarm: geometry visual mesh filename=meshes/elbow_mesh.STL scale=0.005500 0.005500 0.005500; visual mesh filename=meshes/lowerarm_mesh.STL scale=0.006400 0.006400 0.006400
- link right_lowerleg: geometry visual mesh filename=meshes/knee_mesh.STL scale=0.005600 0.005600 0.005600; visual mesh filename=meshes/lowerleg_mesh.STL scale=0.006300 0.006600 0.007000
- link right_upperarm: geometry visual mesh filename=meshes/shoulder_mesh.STL scale=0.003900 0.003900 0.003900; visual mesh filename=meshes/upperarm_mesh.STL scale=0.006300 0.006000 0.006900
- link right_upperleg: geometry visual mesh filename=meshes/upperleg_mesh.STL scale=0.006200 0.006400 0.006900
